File: 3A/load/load.kicad_pcb (KiCad board)
At the start: 4 copper layers, 50 x 50 mm, 56 parts, among them J1 Screw_Terminal_01x02, J2 Screw_Terminal_01x02, Q1 PMBT2222A, Q2 IXTH64N10L2, U1 LMC7660, U2 MCP1501-25xRW, U3 ACS711xLCTR-25AB, U4 OPA2727, U5 TLA2518IRTER, U6 DAC7811IDGST

Commit message: added gerber files
Connections:
- U2 pad 9: (no net) -> GND
Routing:
- net GND: track 51.5 -> 54.6 mm
- net -10V: vias 10 -> 6
