File: 2A/Electronique/Schema Electronique 2223/MainBoard/Intelligence.kicad_sch (KiCad schematic)
At the start: 36 parts, among them J1 Screw_Terminal_01x01, J2 Screw_Terminal_01x01, J3 Screw_Terminal_01x01, J4 Screw_Terminal_01x01, U1 NUCLEO_F446RE

Commit message: schematic and pcb update, added BOM
Parts:
- removed JP4: Jumper_3_Open, Connector_PinHeader_2.54mm:PinHeader_1x03_P2.54mm_Vertical, symbol Jumper:Jumper_3_Open
- D1, D2, D3: value DF3A6.8LFV -> ESD7C5.0DT5G; Mouser Part Number (none) -> 863-ESD7C5.0DT5G
- renumbered UART1 to UART4, UART2 to UART5, UART3 to UART6
Connections:
- net +3.3V: now also R10.1, R9.1
- net CAN1_RX: now also CAN1.1 (Pin_1); no longer CAN1.2 (Pin_2)
- net CAN1_TX: now also CAN1.2 (Pin_2); no longer CAN1.1 (Pin_1)
