File: 2A/Electronique/Schema Electronique 2223/MainBoard/MainBoard.kicad_pcb (KiCad board)
At the start: 2 copper layers, 103.6 x 98.5 mm, 70 parts, among them J1 Screw_Terminal_01x01, J2 Screw_Terminal_01x01, J3 Screw_Terminal_01x01, J4 Screw_Terminal_01x01, M0 Jumper_2_Open, M1 Jumper_2_Open, M2 Jumper_2_Open, Q1 Q_PMOS_GDS, Q2 MBT3906DW1, Q3 PMOS, U1 NUCLEO_F446RE, U4 TSR_1-2450

Commit message: schematic and pcb update, added BOM
Parts:
- D1, D2, D3: value DF3A6.8LFV -> ESD7C5.0DT5G
- D4: value 10V -> 4V7
- D5: value SM6T24A -> 1.5SMBJ36CA
- LED1, LED2, PWR: footprint LED_SMD:LED_0805_2012Metric_Pad1.15x1.40mm_HandSolder -> schematic1:LEDC2012X90N
- Q1: value Q_PMOS_GDS -> PMOS
- R7, R8: footprint Resistor_SMD:R_0805_2012Metric_Pad1.20x1.40mm_HandSolder -> schematic1:R0805
- moved C3 12.2 mm to (96.9, 97.1), turned to 0 degrees
- moved R19 9.70 mm to (97.9, 110.6), turned to 180 degrees
- moved D4 3.61 mm to (98.1, 108.1), turned to 0 degrees
- renumbered ARU to ARU1, M2 to JP10, M0 to JP5, M1 to JP6, M2 to JP7, M0 to JP8, M1 to JP9, L_STEP to LSTEP1, L_ENCODER to L_ENCODER1, PWR_OUT to PWROUT1, R_STEP to RSTEP1, R_ENCODER to R_ENCODER1, L_DRIVER to U2, R_DRIVER to U3, UART1 to UART4, UART2 to UART5, UART3 to UART6
Connections:
- C3 pad +: VBAT -> (no net)
- C3 pad -: GND -> (no net)
Routing:
- net Net-(Q1-G): track 8.57 -> 13.4 mm
- net Net-(D4-A): track 3.79 -> 4.69 mm
- net GND: vias 0 -> 1

Commit message: added vias to pcb
Connections:
- C3 pad +: (no net) -> VBAT
- C3 pad -: (no net) -> GND
Routing:
- net VBAT: track 235.1 -> 235.3 mm, vias 1 -> 37
- net Net-(D5-A2): vias 0 -> 31
- net GND: vias 1 -> 109
- added copper zone on B.Cu, net Net-(D5-A2)
- added copper zone on B.Cu, net VBAT
