File: 2A/Electronique/Schema Electronique 2223/dossier lidar/detection_pcb/detection_pcb.kicad_pcb (KiCad board)
At the start: 2 copper layers, 96 x 96 mm, 142 parts, among them J1 BAT, Q1 PMOS, U1 VL53L1X_module, U10 VL53L1X_module, U11 VL53L1X_module, U12 VL53L1X_module, U13 VL53L1X_module, U14 VL53L1X_module, U15 VL53L1X_module, U16 VL53L1X_module, U17 Buck_3.3V, U18 STM32G070, U2 VL53L1X_module, U3 VL53L1X_module, U4 VL53L1X_module, U5 VL53L1X_module, U6 VL53L1X_module, U7 VL53L1X_module, U8 VL53L1X_module, U9 VL53L1X_module, Y1 16MHz

Commit message: removed duplicated project, updated schematic and pcb, added BOM
Parts:
- added R36: DNP, Resistor_SMD:R_0805_2012Metric, F.Cu at (147.6, 76.2)
- added R37: DNP, Resistor_SMD:R_0805_2012Metric, F.Cu at (150.0, 76.2)
- added RX1: TestPoint, TestPoint:TestPoint_Pad_D1.0mm, B.Cu at (150.0, 77.1)
- added TX1: TestPoint, TestPoint:TestPoint_Pad_D1.0mm, B.Cu at (147.6, 77.1)
- D1: renamed from D2; value 10V -> 4V7
- D2: renamed from D1; value SM6T24A -> 1.5SMBJ36CA
- D3: value NUP2105L -> ESD7C5.0DT5G; footprint Package_TO_SOT_SMD:SOT-23 -> Package_TO_SOT_SMD:SOT-416
- renumbered C2 to C1, C1 to C2, R50 to R34, R51 to R35, R34 to R38, R35 to R39, R36 to R40, R37 to R41, R38 to R42, R39 to R43, R40 to R44, R41 to R45, R42 to R46, R43 to R47, R44 to R48, R45 to R49, R46 to R50, R47 to R51, R48 to R52, R49 to R53, U17 to U1, U9 to U10, U10 to U11, U11 to U12, U12 to U13, U13 to U14, U14 to U15, U15 to U16, U16 to U17, U1 to U2, U2 to U3, U3 to U4, U4 to U5, U5 to U6, U6 to U7, U7 to U8, U8 to U9, XSDN16 to XSDN1, XSDN8 to XSDN11, XSDN4 to XSDN12, XSDN3 to XSDN14, XSDN12 to XSDN15, XSDN2 to XSDN16, XSDN7 to XSDN2, XSDN15 to XSDN3, XSDN11 to XSDN4, XSDN9 to XSDN5, XSDN14 to XSDN6, XSDN1 to XSDN7, XSDN6 to XSDN8, XSDN5 to XSDN9
Routing:
- net +3V3: track 513.3 -> 550.0 mm
- net TX: track 14.1 -> 27.0 mm
- net RX: track 14.2 -> 26.1 mm
- net GND: vias 38 -> 41
