File: 2A/Electronique/Schema Electronique 2223/dossier lidar/detection_pcb/mcu.kicad_sch (KiCad schematic)
At the start: 36 parts, among them U18 STM32G070, Y1 16MHz

Commit message: removed duplicated project, updated schematic and pcb, added BOM
Parts:
- added R52, R53: DNP, Resistor_SMD:R_0805_2012Metric, symbol Device:R_Small
- added RX, TX: TestPoint, TestPoint:TestPoint_Pad_D1.0mm, symbol Connector:TestPoint
- D3: value NUP2105L -> ESD7C5.0DT5G; footprint Package_TO_SOT_SMD:SOT-23 -> Package_TO_SOT_SMD:SOT-416; Mouser Part Number (none) -> 863-ESD7C5.0DT5G
Connections:
- net +3V3: now also R52.1, R53.1
- net RX: now also R52.2, RX.1
- net TX: now also R53.2, TX.1
Other:
- note added: "I2C Pullups"
- note added: "STLINK UART not connected"
- note added: "UART + ESD protection Optionnal pullups"
- moved on the sheet: C22, D3, JP1, SWD1, UART1
