File: 2A/Electronique/Schema Electronique 2223/puissance/puissance.kicad_sch (KiCad schematic)
At the start: 45 parts, among them J1 Conn_01x02, J10 Conn_01x02, J11 Conn_01x02, J12 Conn_01x02, J13 Conn_01x02, J14 Conn_01x03, J15 Conn_01x04, J16 Conn_02x20_Counter_Clockwise, J17 Connecteur bouton Arret Urgen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, J18 Bat 2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

Commit message: data
Parts:
- removed J10, J12, J9: Conn_01x02, symbol Connector_Generic:Conn_01x02
- added J9: Conn_01x04, symbol Connector_Generic:Conn_01x04
Other:
- note added: "Connecteur XL320"
- note added: "Connecteurs 14.4V"
- note added: "Convertion 14.4V vers 7.4V"
- note added: "Pinheader pour effectuer la connection avec la RasberryPi"
- note added: "Verification fonctionnement"
- note removed: "Connecteur Switch alimentation"
- note removed: "Connecteur de lien avec la RasberryPi"
- note removed: "Connecteurs batteries Batteries Nimh 7.2V"
- note removed: "Entree alimentation et Boutton arret Urgence"
- moved on the sheet: D1, D2, H1, H2, H3, H4, J11, J14, J15, J16, J3, J4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
