File: 2A/Electronique/Schema Electronique 2223/puissance/Connectors.kicad_sch (KiCad schematic)
At the start: 35 parts, among them J1 Conn_01x03, J10 Conn_01x03, J11 Conn_01x03, J12 Conn_01x03, J13 Conn_01x05, J14 Conn_01x05, J16 Conn_01x02, J17 Conn_01x02, J18 Conn_01x02, J19 Conn_01x02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

Commit message: add datasheet info
Parts:
- NC7WZ1: Numero de fabrication (none) -> SN74LVC2G241DCTR; nemero mouser (none) -> 595-SN74LVC2G241DCTR
- U1: numero mouser (none) -> 595-SN74LVC2G241DCTR
Changed lines of the file:
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@@
       (effects (font (size 1.27 1.27)) hide)
     )
-    (property "Datasheet" "http://www.ti.com/lit/sg/scyt129e/scyt129e.pdf" (at 76.2282 76.2 0)
+    (property "Datasheet" "https://www.ti.com/lit/ds/symlink/sn74lvc2g241.pdf?ts=1706023484753" (at 76.2282 76.2 0)
+      (effects (font (size 1.27 1.27)) hide)
+    )
+    (property "Numero de fabrication" "SN74LVC2G241DCTR" (at 76.2282 76.2 0)
+      (effects (font (size 1.27 1.27)) hide)
+    )
+    (property "nemero mouser" "595-SN74LVC2G241DCTR" (at 76.2282 76.2 0)
       (effects (font (size 1.27 1.27)) hide)
     )
@@
       (effects (font (size 1.27 1.27)) hide)
     )
-    (property "Datasheet" "http://www.ti.com/lit/sg/scyt129e/scyt129e.pdf" (at 76.2282 47.244 0)
+    (property "Datasheet" "https://www.ti.com/lit/ds/symlink/sn74lvc2g241.pdf?ts=1706023484753" (at 76.2282 47.244 0)
+      (effects (font (size 1.27 1.27)) hide)
+    )
+    (property "numero mouser" "595-SN74LVC2G241DCTR" (at 76.2282 47.244 90)
       (effects (font (size 1.27 1.27)) hide)
     )
@@
       (effects (font (size 1.27 1.27)) hide)
     )
-    (property "Datasheet" "http://www.ti.com/lit/sg/scyt129e/scyt129e.pdf" (at 88.9282 60.96 0)
-      (effects (font (size 1.27 1.27)) hide)
-    )
+    (property "Datasheet" "https://www.ti.com/lit/ds/symlink/sn74lvc2g241.pdf?ts=1706023484753" (at 88.9282 60.96 0)
+      (effects (font (size 1.27 1.27)) hide)
+    )
+    (property "numero mouser" "595-SN74LVC2G241DCTR" (at 88.9282 60.96 90)
+      (effects (font (size 1.27 1.27)) hide)
+    )
