File: 2A/Electronique/Schema Electronique 2223/puissanceok/puissanceok.kicad_sch (KiCad schematic)
At the start: 26 parts, among them J101 Bat 2, J102 Bat 1, J103 AU, J104 Switch, J11 Conn_01x05, J113 Conn_02x20_Odd_Even, J18 Conn_01x02, J19 Conn_01x02, J20 Conn_01x02, J21 Conn_01x02, J7 Conn_01x02, J9 Conn_01x05

Commit message: suppression diode et changement des feuille hiérarchique
Connections:
- net GPIO11: now reaches J113.23 (Pin_23)
- net GPIO2: now reaches J113.3 (Pin_3)
- net GPIO6: now reaches J113.31 (Pin_31)
- net GPIO3: now reaches J113.5 (Pin_5)
- net GPIO35_PWM renamed GPIO19
- net GPIO36 renamed GPIO16
- net GPIO38 renamed GPIO20
- net GPIO40 renamed GPIO21
Other:
- added sheet GPIO_3V3_Connector4 (GPIO_3V3_Connector.kicad_sch)
- added sheet GPIO_3V3_Connector5 (GPIO_3V3_Connector.kicad_sch)
- added sheet GPIO_3V3_Connector6 (GPIO_3V3_Connector.kicad_sch)
- added sheet GPIO_3V3_Connector7 (GPIO_3V3_Connector.kicad_sch)
Changed lines of the file:
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@@
+    (stroke (width 0) (type default))
+  )
+  (wire (pts (xy 271.78 96.52) (xy 275.59 96.52))
     (stroke (width 0) (type default))
   )
@@
     (stroke (width 0) (type default))
   )
+  (wire (pts (xy 271.78 73.66) (xy 275.59 73.66))
+    (stroke (width 0) (type default))
+  )
   (wire (pts (xy 77.47 133.35) (xy 68.58 133.35))
     (stroke (width 0) (type default))
@@
     (stroke (width 0) (type default))
   )
+  (wire (pts (xy 50.8 123.19) (xy 55.88 123.19))
+    (stroke (width 0) (type default))
+  )
   (wire (pts (xy 70.866 49.022) (xy 83.566 49.022))
     (stroke (width 0) (type default))
@@
   )
   (wire (pts (xy 123.19 160.02) (xy 123.19 161.29))
+    (stroke (width 0) (type default))
+  )
+  (wire (pts (xy 271.78 81.28) (xy 275.59 81.28))
+    (stroke (width 0) (type default))
+  )
+  (wire (pts (xy 271.78 88.9) (xy 275.59 88.9))
     (stroke (width 0) (type default))
   )
@@
     (fill (type none))
   )
-  (rectangle (start 233.68 63.5) (end 267.97 101.6)
+  (rectangle (start 233.68 63.5) (end 283.21 101.6)
     (stroke (width 0) (type default))
     (fill (type none))
@@
     (effects (font (size 1.27 1.27) (color 255 191 0 1)) (justify left bottom))
   )
+  (label "GPIO6" (at 50.8 123.19 180) (fields_autoplaced)
+    (effects (font (size 1.27 1.27)) (justify right bottom))
+    (property "info" "pwm" (at 50.8 124.46 0)
+      (effects (font (size 1.27 1.27) italic) (justify right) hide)
+    )
+  )
   (label "Uart4_TX" (at 72.39 113.03 0) (fields_autoplaced)
     (effects (font (size 1.27 1.27) (color 255 0 139 1)) (justify left bottom))
@@
     (effects (font (size 1.27 1.27) (color 255 191 0 1)) (justify left bottom))
   )
-  (label "GPIO40" (at 77.47 133.35 0) (fields_autoplaced)
-    (effects (font (size 1.27 1.27)) (justify left bottom))
+  (label "GPIO3" (at 275.59 81.28 0) (fields_autoplaced)
+    (effects (font (size 1.27 1.27)) (justify left bottom))
+  )
+  (label "GPIO21" (at 77.47 133.35 0) (fields_autoplaced)
+    (effects (font (size 1.27 1.27)) (justify left bottom))
+  )
+  (label "GPIO2" (at 55.88 87.63 180) (fields_autoplaced)
+    (effects (font (size 1.27 1.27)) (justify right bottom))
   )
   (label "FDC_3" (at 123.19 102.87 0) (fields_autoplaced)
     (effects (font (size 1.27 1.27) (color 0 132 0 1)) (justify left bottom))
   )
+  (label "GPIO11" (at 55.88 113.03 180) (fields_autoplaced)
+    (effects (font (size 1.27 1.27)) (justify right bottom))
+  )
   (label "3V3" (at 272.2907 23.426 0) (fields_autoplaced)
     (effects (font (size 1.27 1.27)) (justify left bottom))
@@
     (effects (font (size 1.27 1.27) (color 0 1 255 1)) (justify left bottom))
   )
-  (label "GPIO36" (at 77.47 128.27 0) (fields_autoplaced)
+  (label "GPIO16" (at 77.47 128.27 0) (fields_autoplaced)
     (effects (font (size 1.27 1.27)) (justify left bottom))
   )
@@
     (effects (font (size 1.27 1.27) (color 0 132 0 1)) (justify left bottom))
   )
-  (label "GPIO38" (at 251.46 88.9 0) (fields_autoplaced)
+  (label "GPIO20" (at 251.46 88.9 0) (fields_autoplaced)
     (effects (font (size 1.27 1.27)) (justify left bottom))
   )
@@
     (effects (font (size 1.27 1.27)) (justify left bottom))
   )
-  (label "GPIO38" (at 77.47 130.81 0) (fields_autoplaced)
+  (label "GPIO20" (at 77.47 130.81 0) (fields_autoplaced)
     (effects (font (size 1.27 1.27)) (justify left bottom))
   )
@@
     (effects (font (size 1.27 1.27) (color 250 26 255 1)) (justify left bottom))
   )
+  (label "GPIO6" (at 275.59 96.52 0) (fields_autoplaced)
+    (effects (font (size 1.27 1.27)) (justify left bottom))
+  )
   (label "Uart2_RX" (at 72.39 118.11 0) (fields_autoplaced)
     (effects (font (size 1.27 1.27) (color 255 2 4 1)) (justify left bottom))
@@
     (effects (font (size 1.27 1.27) (color 0 1 255 1)) (justify left bottom))
   )
-  (label "GPIO35_PWM" (at 50.8 128.27 180) (fields_autoplaced)
-    (effects (font (size 1.27 1.27)) (justify right bottom))
-  )
   (label "Uart3_RX" (at 52.07 120.65 180) (fields_autoplaced)
     (effects (font (size 1.27 1.27) (color 255 115 25 1)) (justify right bottom))
@@
     (effects (font (size 1.27 1.27) (color 0 132 0 1)) (justify left bottom))
   )
-  (label "GPIO36" (at 251.46 81.28 0) (fields_autoplaced)
+  (label "GPIO19" (at 251.46 81.28 0) (fields_autoplaced)
     (effects (font (size 1.27 1.27)) (justify left bottom))
   )
@@
     (effects (font (size 1.27 1.27) (color 255 0 139 1)) (justify left bottom))
   )
-  (label "GPIO40" (at 251.46 96.52 0) (fields_autoplaced)
+  (label "GPIO21" (at 251.46 96.52 0) (fields_autoplaced)
     (effects (font (size 1.27 1.27)) (justify left bottom))
   )
@@
     (effects (font (size 1.27 1.27)) (justify left bottom))
   )
-  (label "GPIO35_PWM" (at 251.46 73.66 0) (fields_autoplaced)
-    (effects (font (size 1.27 1.27)) (justify left bottom))
+  (label "GPIO16" (at 251.46 73.66 0) (fields_autoplaced)
+    (effects (font (size 1.27 1.27)) (justify left bottom))
+    (property "info" "pwm" (at 251.46 74.93 0)
+      (effects (font (size 1.27 1.27) italic) (justify left) hide)
+    )
   )
   (label "FDC_3" (at 44.45 102.87 180) (fields_autoplaced)
@@
     (effects (font (size 1.27 1.27) (color 255 115 25 1)) (justify left bottom))
   )
+  (label "GPIO2" (at 275.59 73.66 0) (fields_autoplaced)
+    (effects (font (size 1.27 1.27)) (justify left bottom))
+  )
+  (label "GPIO3" (at 55.88 90.17 180) (fields_autoplaced)
+    (effects (font (size 1.27 1.27)) (justify right bottom))
+  )
   (label "Uart2_RX" (at 217.17 87.63 0) (fields_autoplaced)
     (effects (font (size 1.27 1.27) (color 255 2 4 1)) (justify left bottom))
   )
+  (label "GPIO11" (at 275.59 88.9 0) (fields_autoplaced)
+    (effects (font (size 1.27 1.27)) (justify left bottom))
+  )
   (label "Uart4_TX" (at 217.17 119.38 0) (fields_autoplaced)
     (effects (font (size 1.27 1.27) (color 255 0 139 1)) (justify left bottom))
@@
   (label "Uart1_TX" (at 217.17 78.74 0) (fields_autoplaced)
     (effects (font (size 1.27 1.27) (color 255 191 0 1)) (justify left bottom))
+  )
+  (label "GPIO19" (at 50.8 128.27 180) (fields_autoplaced)
+    (effects (font (size 1.27 1.27)) (justify right bottom))
+    (property "info" "pwm" (at 50.8 129.54 0)
+      (effects (font (size 1.27 1.27) italic) (justify right) hide)
+    )
   )
   (label "3V3" (at 156.21 116.84 0) (fields_autoplaced)
@@
     )
   )
+  (sheet (at 259.08 78.74) (size 12.7 5.08) (fields_autoplaced)
+    (stroke (width 0.1524) (type solid))
+    (fill (color 0 0 0 0.0000))
+    (property "Sheetname" "GPIO_3V3_Connector5" (at 259.08 78.0284 0)
+      (effects (font (size 1.27 1.27)) (justify left bottom))
+    )
+    (property "Sheetfile" "GPIO_3V3_Connector.kicad_sch" (at 259.08 84.4046 0)
+      (effects (font (size 1.27 1.27)) (justify left top) hide)
+    )
+    (pin "Signal" input (at 271.78 81.28 0)
+      (effects (font (size 1.27 1.27)) (justify right))
+    )
+    (instances
+      (project "puissanceok"
+        (path "/50648b18-b1a7-4d76-a5dd-1fad5f3e825e" (page "15"))
+      )
+    )
+  )
+  (sheet (at 259.08 93.98) (size 12.7 5.08) (fields_autoplaced)
+    (stroke (width 0.1524) (type solid))
+    (fill (color 0 0 0 0.0000))
+    (property "Sheetname" "GPIO_3V3_Connector6" (at 259.08 93.2684 0)
+      (effects (font (size 1.27 1.27)) (justify left bottom))
+    )
+    (property "Sheetfile" "GPIO_3V3_Connector.kicad_sch" (at 259.08 99.6446 0)
+      (effects (font (size 1.27 1.27)) (justify left top) hide)
+    )
+    (pin "Signal" input (at 271.78 96.52 0)
+      (effects (font (size 1.27 1.27)) (justify right))
+    )
+    (instances
+      (project "puissanceok"
+        (path "/50648b18-b1a7-4d76-a5dd-1fad5f3e825e" (page "18"))
+      )
+    )
+  )
   (sheet (at 234.95 71.12) (size 12.7 5.08) (fields_autoplaced)
     (stroke (width 0.1524) (type solid))
@@
     )
   )
+  (sheet (at 259.08 86.36) (size 12.7 5.08) (fields_autoplaced)
+    (stroke (width 0.1524) (type solid))
+    (fill (color 0 0 0 0.0000))
+    (property "Sheetname" "GPIO_3V3_Connector7" (at 259.08 85.6484 0)
+      (effects (font (size 1.27 1.27)) (justify left bottom))
+    )
+    (property "Sheetfile" "GPIO_3V3_Connector.kicad_sch" (at 259.08 92.0246 0)
+      (effects (font (size 1.27 1.27)) (justify left top) hide)
+    )
+    (pin "Signal" input (at 271.78 88.9 0)
+      (effects (font (size 1.27 1.27)) (justify right))
+    )
+    (instances
+      (project "puissanceok"
+        (path "/50648b18-b1a7-4d76-a5dd-1fad5f3e825e" (page "17"))
+      )
+    )
+  )
   (sheet (at 234.95 78.74) (size 12.7 5.08) (fields_autoplaced)
     (stroke (width 0.1524) (type solid))
@@
       )
     )
+  )
+  (sheet (at 259.08 71.12) (size 12.7 5.08) (fields_autoplaced)
+    (stroke (width 0.1524) (type solid))
+    (fill (color 0 0 0 0.0000))
+    (property "Sheetname" "GPIO_3V3_Connector4" (at 259.08 70.4084 0)
+      (effects (font (size 1.27 1.27)) (justify left bottom))
+    )
+    (property "Sheetfile" "GPIO_3V3_Connector.kicad_sch" (at 259.08 76.7846 0)
+      (effects (font (size 1.27 1.27)) (justify left top) hide)
+    )
+    (pin "Signal" input (at 271.78 73.66 0)
+      (effects (font (size 1.27 1.27)) (justify right))
+    )
+    (instances
+      (project "puissanceok"
+        (path "/50648b18-b1a7-4d76-a5dd-1fad5f3e825e" (page "16"))
+      )
+    )

Commit message: update schematic add testpoint and level shifter
Parts:
- added TP1: 7.4V, symbol Connector:TestPoint
- added TP2: 5.1V, symbol Connector:TestPoint
- added TP3: TestPoint, symbol Connector:TestPoint
- added TP4: 3V3, symbol Connector:TestPoint
Connections:
- net 3V3: now also TP4.1
- net 5.1V: now also TP2.1
- net 7.4V: now also TP1.1
- net Vin: now also TP3.1
Changed lines of the file:
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@@
   (junction (at 140.716 186.944) (diameter 0) (color 0 0 0 0)
   )
+  (junction (at 272.2907 25.6793) (diameter 0) (color 0 0 0 0)
+  )
   (junction (at 49.276 33.782) (diameter 0) (color 0 0 0 0)
   )
@@
   (junction (at 123.19 160.02) (diameter 0) (color 0 0 0 0)
   )
+  (junction (at 158.1501 36.322) (diameter 0) (color 0 0 0 0)
+  )
   (junction (at 83.566 49.022) (diameter 0) (color 0 0 0 0)
   )
@@
   (junction (at 244.856 121.666) (diameter 0) (color 0 0 0 0)
   )
+  (junction (at 213.3914 36.322) (diameter 0) (color 0 0 0 0)
+  )
   (junction (at 121.92 151.13) (diameter 0) (color 0 0 0 0)
   )
@@
   )
   (junction (at 70.866 33.782) (diameter 0) (color 0 0 0 0)
+  )
+  (junction (at 88.7007 33.782) (diameter 0) (color 0 0 0 0)
   )
   (junction (at 121.92 138.43) (diameter 0) (color 0 0 0 0)
@@
     (stroke (width 0) (type default))
   )
-  (wire (pts (xy 272.2907 23.426) (xy 272.2907 27.236))
+  (wire (pts (xy 272.2907 23.426) (xy 272.2907 25.6793))
     (stroke (width 0) (type default))
   )
@@
     (stroke (width 0) (type default))
   )
-  (wire (pts (xy 211.836 36.322) (xy 215.646 36.322))
-    (stroke (width 0) (type default))
-  )
   (wire (pts (xy 68.326 33.782) (xy 70.866 33.782))
     (stroke (width 0) (type default))
@@
     (stroke (width 0) (type default))
   )
+  (wire (pts (xy 88.7007 33.782) (xy 83.566 33.782))
+    (stroke (width 0) (type default))
+  )
   (wire (pts (xy 68.58 92.71) (xy 72.39 92.71))
     (stroke (width 0) (type default))
@@
     (stroke (width 0) (type default))
   )
-  (wire (pts (xy 154.686 36.322) (xy 161.036 36.322))
+  (wire (pts (xy 211.836 36.322) (xy 213.3914 36.322))
+    (stroke (width 0) (type default))
+  )
+  (wire (pts (xy 154.686 36.322) (xy 158.1501 36.322))
     (stroke (width 0) (type default))
   )
@@
     (stroke (width 0) (type default))
   )
+  (wire (pts (xy 213.3914 36.322) (xy 215.646 36.322))
+    (stroke (width 0) (type default))
+  )
   (wire (pts (xy 52.07 118.11) (xy 55.88 118.11))
     (stroke (width 0) (type default))
@@
     (stroke (width 0) (type default))
   )
+  (wire (pts (xy 272.2907 25.6793) (xy 272.2907 27.236))
+    (stroke (width 0) (type default))
+  )
   (wire (pts (xy 123.19 160.02) (xy 123.19 161.29))
     (stroke (width 0) (type default))
@@
     (stroke (width 0) (type default))
   )
-  (wire (pts (xy 92.456 33.782) (xy 83.566 33.782))
+  (wire (pts (xy 92.456 33.782) (xy 88.7007 33.782))
     (stroke (width 0) (type default))
   )
   (wire (pts (xy 123.19 153.67) (xy 123.19 160.02))
+    (stroke (width 0) (type default))
+  )
+  (wire (pts (xy 158.1501 36.322) (xy 161.036 36.322))
     (stroke (width 0) (type default))
   )
@@
     )
   )
+  (symbol (lib_id "Connector:TestPoint") (at 272.2907 25.6793 90) (unit 1)
+    (in_bom yes) (on_board yes) (dnp no)
+    (property "Reference" "TP4" (at 266.8197 26.7023 0)
+      (effects (font (size 1.27 1.27)) (justify left))
+    )
+    (property "Value" "3V3" (at 268.752 25.111 0)
+      (effects (font (size 1.27 1.27)) (justify left))
+    )
+    (property "Footprint" "" (at 272.2907 20.5993 0)
+      (effects (font (size 1.27 1.27)) hide)
+    )
+    (property "Datasheet" "~" (at 272.2907 20.5993 0)
+      (effects (font (size 1.27 1.27)) hide)
+    )
+    (pin "1")
+    (instances
+      (project "puissanceok"
+        (path "/50648b18-b1a7-4d76-a5dd-1fad5f3e825e"
+          (reference "TP4") (unit 1)
+        )
+      )
+    )
+  )
   (symbol (lib_id "Connector_Generic:Conn_01x02") (at 129.54 160.02 0) (mirror x) (unit 1)
     (in_bom yes) (on_board yes) (dnp no)
@@
     )
   )
+  (symbol (lib_id "Connector:TestPoint") (at 158.1501 36.322 0) (unit 1)
+    (in_bom yes) (on_board yes) (dnp no)
+    (property "Reference" "TP2" (at 157.1271 30.851 0)
+      (effects (font (size 1.27 1.27)) (justify left))
+    )
+    (property "Value" "5.1V" (at 158.7184 32.7833 0)
+      (effects (font (size 1.27 1.27)) (justify left))
+    )
+    (property "Footprint" "" (at 163.2301 36.322 0)
+      (effects (font (size 1.27 1.27)) hide)
+    )
+    (property "Datasheet" "~" (at 163.2301 36.322 0)
+      (effects (font (size 1.27 1.27)) hide)
+    )
+    (pin "1")
+    (instances
+      (project "puissanceok"
+        (path "/50648b18-b1a7-4d76-a5dd-1fad5f3e825e"
+          (reference "TP2") (unit 1)
+        )
+      )
+    )
+  )
   (symbol (lib_id "power:GND") (at 241.046 124.206 0) (unit 1)
     (in_bom yes) (on_board yes) (dnp no)
@@
         (path "/50648b18-b1a7-4d76-a5dd-1fad5f3e825e"
           (reference "J21") (unit 1)
+        )
+      )
+    )
+  )
+  (symbol (lib_id "Connector:TestPoint") (at 88.7007 33.782 0) (unit 1)
+    (in_bom yes) (on_board yes) (dnp no)
+    (property "Reference" "TP3" (at 87.6777 28.311 0)
+      (effects (font (size 1.27 1.27)) (justify left))
+    )
+    (property "Value" "TestPoint" (at 89.269 30.2433 0)
+      (effects (font (size 1.27 1.27)) (justify left))
+    )
+    (property "Footprint" "" (at 93.7807 33.782 0)
+      (effects (font (size 1.27 1.27)) hide)
+    )
+    (property "Datasheet" "~" (at 93.7807 33.782 0)
+      (effects (font (size 1.27 1.27)) hide)
+    )
+    (pin "1")
+    (instances
+      (project "puissanceok"
+        (path "/50648b18-b1a7-4d76-a5dd-1fad5f3e825e"
+          (reference "TP3") (unit 1)
         )
       )
@@
         )
       )
+    )
+  )
+  (symbol (lib_id "Connector:TestPoint") (at 213.3914 36.322 0) (unit 1)
+    (in_bom yes) (on_board yes) (dnp no)
+    (property "Reference" "TP1" (at 212.3684 30.851 0)
+      (effects (font (size 1.27 1.27)) (justify left))
+    )
+    (property "Value" "7.4V" (at 213.9597 32.7833 0)
+      (effects (font (size 1.27 1.27)) (justify left))
+    )
+    (property "Footprint" "" (at 218.4714 36.322 0)
+      (effects (font (size 1.27 1.27)) hide)
+    )
+    (property "Datasheet" "~" (at 218.4714 36.322 0)
+      (effects (font (size 1.27 1.27)) hide)
+    )
+    (pin "1")
+    (instances
+      (project "puissanceok"
+        (path "/50648b18-b1a7-4d76-a5dd-1fad5f3e825e"
+          (reference "TP1") (unit 1)
+        )
+      )
