File: 2A/Electronique/Schema Electronique 2223/puissanceok/XL320.kicad_sch (KiCad schematic)
At the start: 8 parts, among them J21 Conn_XL320, U3 74LVC2G241

Commit message: pcb place components and add power/gnd planes
Parts:
- renumbered C14 to C901, C15 to C902, C16 to C903, J21 to J901, R19 to R901, R21 to R902, R20 to R903, U3 to U901
Changed lines of the file:
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@@
   (symbol (lib_id "power:GND") (at 176.53 111.76 0) (unit 1)
     (in_bom yes) (on_board yes) (dnp no) (fields_autoplaced)
-    (property "Reference" "#PWR050" (at 176.53 118.11 0)
+    (property "Reference" "#PWR0903" (at 176.53 118.11 0)
       (effects (font (size 1.27 1.27)) hide)
     )
@@
       (project "puissanceok"
         (path "/50648b18-b1a7-4d76-a5dd-1fad5f3e825e/6ae65ced-862a-45db-8236-045925bae1ca"
-          (reference "#PWR050") (unit 1)
+          (reference "#PWR0903") (unit 1)
         )
       )
@@
   (symbol (lib_id "Connector_Generic:Conn_01x03") (at 182.88 107.95 0) (mirror x) (unit 1)
     (in_bom yes) (on_board yes) (dnp no)
-    (property "Reference" "J21" (at 185.42 109.22 0)
+    (property "Reference" "J901" (at 185.42 109.22 0)
       (effects (font (size 1.27 1.27)) (justify left))
     )
@@
       (project "puissanceok"
         (path "/50648b18-b1a7-4d76-a5dd-1fad5f3e825e/6ae65ced-862a-45db-8236-045925bae1ca"
-          (reference "J21") (unit 1)
+          (reference "J901") (unit 1)
         )
       )
@@
   (symbol (lib_id "Device:C_Small") (at 201.93 66.04 0) (unit 1)
     (in_bom yes) (on_board yes) (dnp no)
-    (property "Reference" "C16" (at 203.708 65.024 0)
+    (property "Reference" "C903" (at 203.708 65.024 0)
       (effects (font (size 1.27 1.27)) (justify left))
     )
@@
       (project "puissanceok"
         (path "/50648b18-b1a7-4d76-a5dd-1fad5f3e825e/6ae65ced-862a-45db-8236-045925bae1ca"
-          (reference "C16") (unit 1)
+          (reference "C903") (unit 1)
         )
       )
@@
   (symbol (lib_id "74xGxx:74LVC2G241") (at 105.41 69.85 180) (unit 1)
     (in_bom yes) (on_board yes) (dnp no) (fields_autoplaced)
-    (property "Reference" "U3" (at 106.68 58.42 0)
+    (property "Reference" "U901" (at 106.68 58.42 0)
       (effects (font (size 1.27 1.27)))
     )
@@
       (project "puissanceok"
         (path "/50648b18-b1a7-4d76-a5dd-1fad5f3e825e/6ae65ced-862a-45db-8236-045925bae1ca"
-          (reference "U3") (unit 1)
+          (reference "U901") (unit 1)
         )
       )
@@
   (symbol (lib_id "Device:C_Small") (at 175.5932 64.0011 0) (unit 1)
     (in_bom yes) (on_board yes) (dnp no)
-    (property "Reference" "C14" (at 177.8 62.23 0)
+    (property "Reference" "C901" (at 177.8 62.23 0)
       (effects (font (size 1.27 1.27)) (justify left))
     )
@@
       (project "puissanceok"
         (path "/50648b18-b1a7-4d76-a5dd-1fad5f3e825e/6ae65ced-862a-45db-8236-045925bae1ca"
-          (reference "C14") (unit 1)
+          (reference "C901") (unit 1)
         )
       )
@@
   (symbol (lib_id "Device:R_Small") (at 87.63 64.77 0) (unit 1)
     (in_bom yes) (on_board yes) (dnp no) (fields_autoplaced)
-    (property "Reference" "R19" (at 89.408 64.135 0)
+    (property "Reference" "R901" (at 89.408 64.135 0)
       (effects (font (size 1.27 1.27)) (justify left))
     )
@@
       (project "puissanceok"
         (path "/50648b18-b1a7-4d76-a5dd-1fad5f3e825e/6ae65ced-862a-45db-8236-045925bae1ca"
-          (reference "R19") (unit 1)
+          (reference "R901") (unit 1)
         )
       )
@@
   (symbol (lib_id "power:GND") (at 196.85 69.85 0) (unit 1)
     (in_bom yes) (on_board yes) (dnp no) (fields_autoplaced)
-    (property "Reference" "#PWR047" (at 196.85 76.2 0)
+    (property "Reference" "#PWR0904" (at 196.85 76.2 0)
       (effects (font (size 1.27 1.27)) hide)
     )
@@
       (project "puissanceok"
         (path "/50648b18-b1a7-4d76-a5dd-1fad5f3e825e/6ae65ced-862a-45db-8236-045925bae1ca"
-          (reference "#PWR047") (unit 1)
+          (reference "#PWR0904") (unit 1)
         )
       )
@@
   (symbol (lib_id "power:GND") (at 167.64 74.93 0) (unit 1)
     (in_bom yes) (on_board yes) (dnp no)
-    (property "Reference" "#PWR048" (at 167.64 81.28 0)
+    (property "Reference" "#PWR0902" (at 167.64 81.28 0)
       (effects (font (size 1.27 1.27)) hide)
     )
@@
       (project "puissanceok"
         (path "/50648b18-b1a7-4d76-a5dd-1fad5f3e825e/6ae65ced-862a-45db-8236-045925bae1ca"
-          (reference "#PWR048") (unit 1)
+          (reference "#PWR0902") (unit 1)
         )
       )
@@
   (symbol (lib_id "74xGxx:74LVC2G241") (at 107.95 93.98 0) (unit 2)
     (in_bom yes) (on_board yes) (dnp no) (fields_autoplaced)
-    (property "Reference" "U3" (at 106.68 102.87 0)
+    (property "Reference" "U901" (at 106.68 102.87 0)
       (effects (font (size 1.27 1.27)))
     )
@@
       (project "puissanceok"
         (path "/50648b18-b1a7-4d76-a5dd-1fad5f3e825e/6ae65ced-862a-45db-8236-045925bae1ca"
-          (reference "U3") (unit 2)
+          (reference "U901") (unit 2)
         )
       )
@@
   (symbol (lib_id "power:GND") (at 93.98 87.884 0) (unit 1)
     (in_bom yes) (on_board yes) (dnp no)
-    (property "Reference" "#PWR049" (at 93.98 94.234 0)
+    (property "Reference" "#PWR0901" (at 93.98 94.234 0)
       (effects (font (size 1.27 1.27)) hide)
     )
@@
       (project "puissanceok"
         (path "/50648b18-b1a7-4d76-a5dd-1fad5f3e825e/6ae65ced-862a-45db-8236-045925bae1ca"
-          (reference "#PWR049") (unit 1)
+          (reference "#PWR0901") (unit 1)
         )
       )
@@
   (symbol (lib_id "Device:R_Small") (at 93.98 85.09 0) (unit 1)
     (in_bom yes) (on_board yes) (dnp no) (fields_autoplaced)
-    (property "Reference" "R21" (at 95.758 84.455 0)
+    (property "Reference" "R902" (at 95.758 84.455 0)
       (effects (font (size 1.27 1.27)) (justify left))
     )
@@
       (project "puissanceok"
         (path "/50648b18-b1a7-4d76-a5dd-1fad5f3e825e/6ae65ced-862a-45db-8236-045925bae1ca"
-          (reference "R21") (unit 1)
+          (reference "R902") (unit 1)
         )
       )
@@
   (symbol (lib_id "74xGxx:74LVC2G241") (at 167.64 64.77 0) (unit 3)
     (in_bom yes) (on_board yes) (dnp no)
-    (property "Reference" "U3" (at 158.75 66.04 90)
+    (property "Reference" "U901" (at 158.75 66.04 90)
       (effects (font (size 1.27 1.27)) (justify left))
     )
@@
       (project "puissanceok"
         (path "/50648b18-b1a7-4d76-a5dd-1fad5f3e825e/6ae65ced-862a-45db-8236-045925bae1ca"
-          (reference "U3") (unit 3)
+          (reference "U901") (unit 3)
         )
       )
@@
   (symbol (lib_id "Device:R_Small") (at 121.92 66.04 0) (unit 1)
     (in_bom yes) (on_board yes) (dnp no) (fields_autoplaced)
-    (property "Reference" "R20" (at 124.46 64.77 0)
+    (property "Reference" "R903" (at 124.46 64.77 0)
       (effects (font (size 1.27 1.27)) (justify left))
     )
@@
       (project "puissanceok"
         (path "/50648b18-b1a7-4d76-a5dd-1fad5f3e825e/6ae65ced-862a-45db-8236-045925bae1ca"
-          (reference "R20") (unit 1)
+          (reference "R903") (unit 1)
         )
       )
@@
   (symbol (lib_id "Device:C_Polarized_Small") (at 191.77 66.04 0) (unit 1)
     (in_bom yes) (on_board yes) (dnp no) (fields_autoplaced)
-    (property "Reference" "C15" (at 194.31 64.2239 0)
+    (property "Reference" "C902" (at 194.31 64.2239 0)
       (effects (font (size 1.27 1.27)) (justify left))
     )
@@
       (project "puissanceok"
         (path "/50648b18-b1a7-4d76-a5dd-1fad5f3e825e/6ae65ced-862a-45db-8236-045925bae1ca"
-          (reference "C15") (unit 1)
-        )
-      )
+          (reference "C902") (unit 1)
+        )
+      )
