File: 2A/Electronique/Schema Electronique 2223/puissanceok/puissanceok.kicad_pcb (KiCad board)
At the start: 4 copper layers, 66 x 57 mm, 83 parts, among them J1001 Conn_UART, J101 Bat 2, J102 Bat 1, J103 AU, J104 Switch, J105 Conn_RPI, J106 Conn_Phidget_PS_Stepper_1, J107 Conn_Phidget_PS_Stepper_2, J108 Conn_Phidget_PS_Stepper_3, J109 Conn_Phidget_PS_Stepper_4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

Commit message: update errors
Parts:
- removed ?: , 
- removed H104: MountingHole_Pad, MountingHole:MountingHole_2.7mm_M2.5_Pad_Via
- added H103: MountingHole_Pad, MountingHole:MountingHole_2.7mm_M2.5_Pad_Via, F.Cu at (49.9, 99.4)
Routing:
- net 5.1V: track 123.4 -> 117.2 mm, vias 18 -> 17
- net 14.4V: track 54.0 -> 57.7 mm
- net /Out_color_sensor: track 77.6 -> 76.4 mm
- net /GPIO2: track 112.1 -> 113.3 mm
- net /FDC_1: track 61.7 -> 62.7 mm
- net /FDC_2: track 46.9 -> 47.8 mm
- net /GPIO3: track 117.1 -> 118.0 mm
- net GND: track 8.78 -> 8.07 mm
- net /FDC_4: track 42.3 -> 41.6 mm
- net +3.3V: track 47.0 -> 46.3 mm
- net Net-(J401-Pin_2): track 4.69 -> 5.23 mm

Commit message: update pcbpuissance
Routing:
- net GND: vias 29 -> 28
Changed lines of the file:
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@@
   (via (at 103.8 53.3) (size 0.6) (drill 0.25) (layers "F.Cu" "B.Cu") (net 2))
   (via (at 67.8 69.1) (size 0.6) (drill 0.25) (layers "F.Cu" "B.Cu") (net 2))
-  (via (at 90.4 64.4) (size 0.6) (drill 0.25) (layers "F.Cu" "B.Cu") (net 2))
+  (via (at 90.5995 64.4) (size 0.6) (drill 0.25) (layers "F.Cu" "B.Cu") (net 2))
   (via (at 74.5 69) (size 0.6) (drill 0.25) (layers "F.Cu" "B.Cu") (net 2))
-  (via (at 67.7 64.7) (size 0.6) (drill 0.25) (layers "F.Cu" "B.Cu") (net 2))
   (via (at 47.5 88.8) (size 0.6) (drill 0.25) (layers "F.Cu" "B.Cu") (net 2))
   (via (at 78.5 55.5) (size 0.6) (drill 0.25) (layers "F.Cu" "B.Cu") (net 2))
@@
   (via (at 88 97.2) (size 0.6) (drill 0.25) (layers "F.Cu" "B.Cu") (net 24))
   (via (at 81.35 53.65) (size 0.6) (drill 0.25) (layers "F.Cu" "B.Cu") (net 24))
-  (segment (start 89.8 62.1) (end 81.35 53.65) (width 0.2) (layer "B.Cu") (net 24))
-  (segment (start 89.8 95.4) (end 89.8 62.1) (width 0.2) (layer "B.Cu") (net 24))
-  (segment (start 88 97.2) (end 89.8 95.4) (width 0.2) (layer "B.Cu") (net 24))
+  (segment (start 90 95.2) (end 90 62.3) (width 0.2) (layer "B.Cu") (net 24))
+  (segment (start 88 97.2) (end 90 95.2) (width 0.2) (layer "B.Cu") (net 24))
+  (segment (start 90 62.3) (end 81.35 53.65) (width 0.2) (layer "B.Cu") (net 24))
   (segment (start 96.2 91.8) (end 94.9 93.1) (width 0.2) (layer "F.Cu") (net 25))
   (segment (start 96.2 83.15) (end 96.2 91.8) (width 0.2) (layer "F.Cu") (net 25))

Commit message: suppr redflag
Parts:
- moved D601 0.07 mm to (73.9, 56.2)
- moved U601 0.07 mm to (69.4, 68.8)
- moved C602 0.07 mm to (57.5, 72.0)
- moved C603 0.07 mm to (58.0, 68.5)
- moved C604 0.07 mm to (60.0, 56.1)
- moved L601 0.07 mm to (67.5, 58.0)
- moved R601 0.07 mm to (58.5, 72.1)
- moved R602 0.07 mm to (58.0, 70.5)
- moved C601 0.07 mm to (61.8, 78.2)
- moved C605 0.07 mm to (60.0, 61.0)
- moved R603 0.07 mm to (58.1, 69.6)
Routing:
- net 5.1V: track 117.2 -> 123.3 mm
- net +3.3V: track 46.3 -> 48.8 mm
- net 14.4V: track 57.7 -> 60.2 mm, vias 44 -> 43
- net /FDC_1: track 62.7 -> 63.7 mm

Commit message: suppr warning
Parts:
- moved U901 0.35 mm to (103.5, 54.6)
Routing:
- net GND: track 8.40 -> 13.9 mm
- net 14.4V: track 60.2 -> 65.6 mm
Other:
- board text added: "2"
- board text added: "3"
