File: 2A/Electronique/Schema Electronique 2223/puissanceok/puissanceok.kicad_pcb (KiCad board)
At the start: 4 copper layers, 66 x 57 mm, 82 parts, among them J1001 Conn_UART, J101 Bat 2, J102 Bat 1, J103 AU, J104 Switch, J105 Conn_RPI, J106 Conn_Phidget_PS_Stepper_1, J107 Conn_Phidget_PS_Stepper_2, J108 Conn_Phidget_PS_Stepper_3, J109 Conn_Phidget_PS_Stepper_4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

Commit message: update pcb
Routing:
- net /BUCK_7.4V/voutbuck: track 16.7 -> 0.00 mm
- net /BUCK_5.1V/voutbuck: vias 16 -> 0
- added copper zone on F.Cu, net /BUCK_5.1V/voutbuck
- added copper zone on F.Cu, net /BUCK_7.4V/voutbuck
- removed copper zone on B.Cu, net /BUCK_5.1V/voutbuck
Changed lines of the file:
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@@
   (segment (start 107.71 94.1) (end 107.71 94.6025) (width 0.2) (layer "F.Cu") (net 42))
   (segment (start 107.71 94.6025) (end 107.0125 95.3) (width 0.2) (layer "F.Cu") (net 42))
-  (segment (start 84.6 63.18) (end 87.125 60.655) (width 0.2) (layer "F.Cu") (net 43))
-  (segment (start 91.105 60.655) (end 93.455 58.305) (width 0.2) (layer "F.Cu") (net 43))
-  (segment (start 81.35 65.915) (end 84.285 65.915) (width 0.2) (layer "F.Cu") (net 43))
-  (segment (start 84.285 65.915) (end 84.6 65.6) (width 0.2) (layer "F.Cu") (net 43))
-  (segment (start 84.6 65.6) (end 84.6 63.18) (width 0.2) (layer "F.Cu") (net 43))
-  (segment (start 87.125 60.655) (end 91.105 60.655) (width 0.2) (layer "F.Cu") (net 43))
   (segment (start 53.9 67.35) (end 53.9 72.25) (width 0.2) (layer "B.Cu") (net 44))
-  (via (at 60 66.35) (size 0.6) (drill 0.3) (layers "F.Cu" "B.Cu") (net 45))
-  (via (at 73.9 58.8) (size 0.6) (drill 0.3) (layers "F.Cu" "B.Cu") (net 45))
-  (via (at 60.95 66.35) (size 0.6) (drill 0.3) (layers "F.Cu" "B.Cu") (net 45))
-  (via (at 62.85 66.35) (size 0.6) (drill 0.3) (layers "F.Cu" "B.Cu") (net 45))
-  (via (at 61.9 66.35) (size 0.6) (drill 0.3) (layers "F.Cu" "B.Cu") (net 45))
-  (via (at 66.1 61.7) (size 0.6) (drill 0.3) (layers "F.Cu" "B.Cu") (net 45))
-  (via (at 67.25 60.55) (size 0.6) (drill 0.3) (layers "F.Cu" "B.Cu") (net 45))
-  (via (at 70.8 61.65) (size 0.6) (drill 0.3) (layers "F.Cu" "B.Cu") (net 45))
-  (via (at 74.8 60.4) (size 0.6) (drill 0.3) (layers "F.Cu" "B.Cu") (net 45))
-  (via (at 73.1 57.1) (size 0.6) (drill 0.3) (layers "F.Cu" "B.Cu") (net 45))
-  (via (at 68.5 61.7) (size 0.6) (drill 0.3) (layers "F.Cu" "B.Cu") (net 45))
-  (via (at 73.1 60.4) (size 0.6) (drill 0.3) (layers "F.Cu" "B.Cu") (net 45))
-  (via (at 63.75 66.35) (size 0.6) (drill 0.3) (layers "F.Cu" "B.Cu") (net 45))
-  (via (at 69.7 60.6) (size 0.6) (drill 0.3) (layers "F.Cu" "B.Cu") (net 45))
-  (via (at 64.95 60.5) (size 0.6) (drill 0.3) (layers "F.Cu" "B.Cu") (net 45))
-  (via (at 74.9 57.1) (size 0.6) (drill 0.3) (layers "F.Cu" "B.Cu") (net 45))
   (segment (start 53.9 58.95) (end 53.9 63.85) (width 0.2) (layer "B.Cu") (net 46))
   (segment (start 53.9 75.75) (end 53.9 80.65) (width 0.2) (layer "B.Cu") (net 47))
@@
   (segment (start 58.76 71.44) (end 58.6 71.6) (width 0.2) (layer "F.Cu") (net 53))
   (segment (start 61.665 71.6) (end 61.825 71.44) (width 0.2) (layer "F.Cu") (net 53))
+  (zone (net 45) (net_name "/BUCK_5.1V/voutbuck") (layer "F.Cu") (hatch edge 0.5)
+    (priority 5)
+    (connect_pads yes (clearance 0.2))
+    (min_thickness 0.25) (filled_areas_thickness no)
+    (fill yes (thermal_gap 0.5) (thermal_bridge_width 0.5) (smoothing fillet) (radius 0.25))
+    (polygon
+      (pts
+        (xy 72.25 56.1)
+        (xy 72.1 59.8)
+        (xy 63.75 59.75)
+        (xy 63.8 62.4)
+        (xy 63.75 62.5)
+        (xy 58.8 64.3)
+        (xy 58.8 65.85)
+        (xy 58.8 66.85)
+        (xy 64.55 66.9)
+        (xy 76 61.65)
+        (xy 75.95 56.1)
+      )
+    )
+  )
+  (zone (net 43) (net_name "/BUCK_7.4V/voutbuck") (layer "F.Cu") (hatch edge 0.5)
+    (priority 4)
+    (connect_pads yes (clearance 0.2))
+    (min_thickness 0.25) (filled_areas_thickness no)
+    (fill yes (thermal_gap 0.5) (thermal_bridge_width 0.5) (smoothing fillet) (radius 0.25))
+    (polygon
+      (pts
+        (xy 91.5 55.75)
+        (xy 91.5 58.95)
+        (xy 91.2 59.25)
+        (xy 83.1 59.25)
+        (xy 83.1 61.95)
+        (xy 82 63.05)
+        (xy 79.2 63.05)
+        (xy 77.95 64.3)
+        (xy 77.95 66.55)
+        (xy 78.05 66.65)
+        (xy 83.85 66.65)
+        (xy 87.5 63)
+        (xy 93.2 63)
+        (xy 95.45 60.75)
+        (xy 95.45 55.65)
+        (xy 91.6 55.65)
+      )
+    )
+  )
   (zone (net 2) (net_name "GND") (layers "F.Cu" "In1.Cu" "B.Cu") (name "GND") (hatch edge 0.5)
     (connect_pads yes (clearance 0.5))
@@
       )
     )
-  )
-  (zone (net 45) (net_name "/BUCK_5.1V/voutbuck") (layer "B.Cu") (hatch edge 0.5)
-    (priority 10)
-    (connect_pads (clearance 0.2))
-    (min_thickness 0.25) (filled_areas_thickness no)
-    (fill yes (thermal_gap 0.5) (thermal_bridge_width 0.5))
-    (polygon
-      (pts
-        (xy 72.25 56.1)
-        (xy 72.1 59.8)
-        (xy 63.75 59.9)
-        (xy 63.8 62.4)
-        (xy 71.45 62.5)
-        (xy 64.4 65.7)
-        (xy 59.4 65.85)
-        (xy 59.4 66.85)
-        (xy 64.55 66.9)
-        (xy 76 61.65)
-        (xy 75.95 56.1)
-      )
-    )

Commit message: update pcb
Routing:
- net /GPIO3: track 118.0 -> 122.7 mm
- net /FDC_1: track 63.7 -> 68.3 mm
- net 5.1V: track 123.3 -> 125.6 mm
- net /S1_color_sensor: track 63.2 -> 62.1 mm
- net /FDC_2: track 48.3 -> 49.1 mm
- net /S3_color_sensor: track 56.7 -> 55.8 mm
- net GND: vias 28 -> 107
- added copper zone on F.Cu, net 5.1V

Commit message: update pcb
Routing:
- net /S3_color_sensor: track 55.8 -> 70.1 mm
- net /FDC_4: track 41.6 -> 53.2 mm
- net /S2_color_sensor: track 62.8 -> 74.0 mm
- net /S1_color_sensor: track 62.1 -> 69.6 mm
- net 7.4V: track 46.7 -> 47.4 mm, vias 8 -> 22
- added copper zone on F.Cu, net 7.4V
