File: 2A/Electronique/Schema Electronique 2223/puissanceok_papazoglou/puissanceok.kicad_pcb (KiCad board)
At the start: 4 copper layers, 66 x 57 mm, 82 parts, among them J1001 Conn_UART, J101 Bat 2, J102 Bat 1, J103 AU, J104 Switch, J105 Conn_RPI, J106 Conn_Phidget_PS_Stepper_1, J107 Conn_Phidget_PS_Stepper_2, J108 Conn_Phidget_PS_Stepper_3, J109 Conn_Phidget_PS_Stepper_4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

Commit message: add other version of pcb
Connections:
- J105 pad 1: +3.3V -> unconnected-(J105-Pin_1-Pad1)
Changed lines of the file:
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@@
   (net 54 "unconnected-(U301-Ilim-Pad3)")
   (net 55 "unconnected-(U601-Ilim-Pad3)")
+  (net 56 "unconnected-(J105-Pin_1-Pad1)")
   (footprint "Capacitor_SMD:CP_Elec_6.3x7.7" (layer "F.Cu")
     (at 99.2 59.5 -90)
@@
       (stroke (width 0.1) (type solid)) (layer "B.Fab"))
     (pad "1" thru_hole rect (at 0 0 270) (size 1.7 1.7) (drill 1) (layers "*.Cu" "*.Mask")
-      (net 6 "+3.3V") (pinfunction "Pin_1") (pintype "passive"))
+      (net 56 "unconnected-(J105-Pin_1-Pad1)") (pinfunction "Pin_1") (pintype "passive+no_connect"))
     (pad "2" thru_hole oval (at -2.54 0 270) (size 1.7 1.7) (drill 1) (layers "*.Cu" "*.Mask")
       (net 16 "5.1V") (pinfunction "Pin_2") (pintype "passive"))

Commit message: update pcb
Parts:
- moved R901 5.78 mm to (101.9, 52.8), turned to 0 degrees
Connections:
- J105 pad 11: /FDC_1 -> /FDC_3
- J105 pad 13: /FDC_2 -> /FDC_4
- J105 pad 15: /FDC_3 -> /S3_color_sensor
- J105 pad 16: /S0_color_sensor -> /Out_color_sensor
- J105 pad 18: /S1_color_sensor -> /S2_color_sensor
- J105 pad 19: /FDC_4 -> /S1_color_sensor
- J105 pad 22: /S2_color_sensor -> /S0_color_sensor
- J105 pad 23: /GPIO11 -> /GPIO2
- J105 pad 26: /S3_color_sensor -> /GPIO11
- J105 pad 3: /GPIO2 -> /FDC_1
- J105 pad 31: /GPIO6 -> /GPIO3
- J105 pad 35: /GPIO19 -> /GPIO6
- J105 pad 37: /Out_color_sensor -> /GPIO19
- J105 pad 5: /GPIO3 -> /FDC_2
- J112 pad 3: /GPIO6 -> /GPIO11
- J112 pad 4: /GPIO11 -> /GPIO6
Routing:
- net /Out_color_sensor: track 0.00 -> 68.9 mm
- net /S3_color_sensor: track 0.00 -> 64.2 mm
- net /S2_color_sensor: track 0.00 -> 60.1 mm
- net /S0_color_sensor: track 0.00 -> 56.4 mm
- net /S1_color_sensor: track 0.00 -> 54.6 mm
- net /Uart3_TX: track 21.0 -> 65.6 mm, vias 0 -> 1
- net /Uart1_TX: track 5.61 -> 44.7 mm
- net /UartTX_Enable: track 7.65 -> 43.9 mm, vias 0 -> 2
- net /Uart1_RX: track 3.93 -> 39.7 mm
- net /Uart4_TX: track 30.5 -> 64.4 mm, vias 0 -> 1
- net /GPIO11: track 17.6 -> 48.1 mm
- net /GPIO2: track 24.3 -> 52.0 mm
- net /Uart4_RX: track 29.5 -> 56.0 mm
- net /Uart2_RX: track 38.1 -> 58.8 mm, vias 0 -> 1
- net /Uart3_RX: track 22.3 -> 41.5 mm
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
Commit message: vias
Routing:
- net GND: vias 158 -> 323

Commit message: update pcb
Connections:
- J105 pad 23: /GPIO2 -> /GPIO11
- J105 pad 26: /GPIO11 -> /GPIO7
- J105 pad 31: /GPIO3 -> /GPIO6
- J105 pad 35: /GPIO6 -> /GPIO19
- J105 pad 37: /GPIO19 -> /GPIO26
- J112 pad 1: /GPIO2 -> /GPIO11
- J112 pad 2: /GPIO3 -> /GPIO6
- J112 pad 3: /GPIO11 -> /GPIO7
- J112 pad 4: /GPIO6 -> /GPIO19
- J112 pad 6: /GPIO19 -> /GPIO26
Routing:
- net /GPIO2: track 52.0 -> 0.00 mm
- net /GPIO7: track 0.00 -> 48.1 mm
- net /GPIO3: track 36.9 -> 0.00 mm
- net /GPIO26: track 0.00 -> 24.2 mm
- net /GPIO6: track 29.6 -> 36.9 mm
- net /GPIO19: track 24.3 -> 29.6 mm
- net /GPIO11: track 48.1 -> 52.0 mm
- net GND: track 7.32 -> 7.03 mm, vias 323 -> 279

Commit message: update pcb
Parts:
- added G***: LOGO, libs:ares_logo_8mm, F.Cu at (99.7, 70.8)
- added G***: LOGO, libs:ares_ENSEA_8mm, F.Cu at (98.0, 79.5)
Other:
- board text added: "26"
- board text added: "7"
- board text added: "Connector 5.1v"
