File: 2A/Electronique/Schema Electronique 2223/puissanceok_papazoglou/puissanceok.kicad_pcb (KiCad board)
At the start: 4 copper layers, 66 x 57 mm, 84 parts, among them J1001 Conn_UART, J101 Bat 2, J102 Bat 1, J103 AU, J104 Switch, J105 Conn_RPI, J106 Conn_Phidget_PS_Stepper_1, J107 Conn_Phidget_PS_Stepper_2, J108 Conn_Phidget_PS_Stepper_3, J109 Conn_Phidget_PS_Stepper_4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

Commit message: finalize pcb
Parts:
- moved G*** 11.8 mm to (90.8, 78.5), turned to 0 degrees
- moved J108 0.50 mm to (67.0, 93.1)
- moved J109 0.50 mm to (67.0, 99.4)
- moved G*** 0.43 mm to (98.2, 79.1), turned to 0 degrees
Connections:
- J114 pad 1: +3.3V -> GND
- J114 pad 2: GND -> 5.1V
- J114 pad 4: 5.1V -> GND
- J114 pad 5: GND -> +3.3V
Routing:
- net 5.1V: track 122.8 -> 126.5 mm
- net GND: track 7.03 -> 7.49 mm, vias 279 -> 326
Other:
- board text added: "5.1v"
- board text added: "CFR 2024"
- board text added: "Phidget_PS_Stepper ↓↑"
- board text added: "UART 2/4/3"
- board text removed: "Conn_Phidget_PS_Stepper"
- board text removed: "Connector 5.1v"

Commit message: update pcb
Parts:
- added R1: 2k7, Resistor_SMD:R_0402_1005Metric, F.Cu at (104.5, 61.4)
- added R2: 3k3, Resistor_SMD:R_0402_1005Metric, F.Cu at (104.5, 60.4)
- added R3: 2k7, Resistor_SMD:R_0402_1005Metric, F.Cu at (104.5, 63.4)
- added R4: 3k3, Resistor_SMD:R_0402_1005Metric, F.Cu at (104.5, 62.4)
- moved C903 0.51 mm to (104.5, 58.8), turned to 180 degrees
Connections:
- J112 pad 7: /GPIO20 -> Net-(J112-Pin_7)
- J112 pad 8: /GPIO21 -> Net-(J112-Pin_8)
- J113 pad 7: +3.3V -> 7.4V
- J113 pad 8: +3.3V -> 7.4V
Routing:
- net Net-(J112-Pin_7): track 0.00 -> 5.97 mm
- net Net-(J112-Pin_8): track 0.00 -> 5.66 mm
- net 7.4V: track 48.6 -> 53.7 mm
- net /GPIO21: track 18.9 -> 14.5 mm, vias 0 -> 1
- net /GPIO20: track 23.6 -> 20.1 mm, vias 0 -> 1
- net GND: track 7.49 -> 11.0 mm, vias 326 -> 324
Other:
- board text added: "7.4v"
