File: 2A/Electronique/Schema Electronique 2223/puissanceok_papazoglou/XL320.kicad_sch (KiCad schematic)
At the start: 8 parts, among them J901 Conn_XL320, U901 74LVC2G241

Commit message: minimal changes, components
Parts:
- U901: MPN (none) -> 74LVC2G241DC,125
Changed lines of the file:
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@@
+      (effects (font (size 1.27 1.27)) hide)
+    )
+    (property "MPN" "74LVC2G241DC,125" (at 105.41 69.85 0)
       (effects (font (size 1.27 1.27)) hide)
     )
@@
       (effects (font (size 1.27 1.27)) hide)
     )
+    (property "MPN" "74LVC2G241DC,125" (at 107.95 93.98 0)
+      (effects (font (size 1.27 1.27)) hide)
+    )
     (pin "1")
     (pin "2")
@@
       (effects (font (size 1.27 1.27)) hide)
     )
+    (property "MPN" "74LVC2G241DC,125" (at 167.64 64.77 0)
+      (effects (font (size 1.27 1.27)) hide)
+    )
