File: 2A/Electronique/Schema Electronique 2223/puissanceok_papazoglou/puissanceok.kicad_sch (KiCad schematic)
At the start: 33 parts, among them J106 Conn_Phidget_PS_Stepper_1, J107 Conn_Phidget_PS_Stepper_2, J108 Conn_Phidget_PS_Stepper_3, J109 Conn_Phidget_PS_Stepper_4, J110 Conn_01x02, J111 Conn_GND, J112 Conn_GPIO_unused, J113 Conn_3.3V, J114 Conn_01x05, J115 Conn_01x05

Commit message: update pcb
Connections:
- net FDC_1: now also J?.3 (Pin_3); no longer J?.11 (Pin_11)
- net FDC_2: now also J?.5 (Pin_5); no longer J?.13 (Pin_13)
- net FDC_3: now also J?.11 (Pin_11); no longer J?.15 (Pin_15)
- net FDC_4: now also J?.13 (Pin_13); no longer J?.19 (Pin_19)
- net GPIO11: now also J112.3 (Pin_3), J?.26 (Pin_26); no longer J112.4 (Pin_4), J?.23 (Pin_23)
- net GPIO19: now also J?.37 (Pin_37); no longer J?.35 (Pin_35)
- net GPIO2: now also J?.23 (Pin_23); no longer J?.3 (Pin_3)
- net GPIO3: now also J?.31 (Pin_31); no longer J?.5 (Pin_5)
- net GPIO6: now also J112.4 (Pin_4), J?.35 (Pin_35); no longer J112.3 (Pin_3), J?.31 (Pin_31)
- net Out_color_sensor: now also J?.16 (Pin_16); no longer J?.37 (Pin_37)
- net S0_color_sensor: now also J?.22 (Pin_22); no longer J?.16 (Pin_16)
- net S1_color_sensor: now also J?.19 (Pin_19); no longer J?.18 (Pin_18)
- net S2_color_sensor: now also J?.18 (Pin_18); no longer J?.22 (Pin_22)
- net S3_color_sensor: now also J?.15 (Pin_15); no longer J?.26 (Pin_26)

Commit message: update pcb
Connections:
- net GPIO2 is gone; now on net GPIO11: J112.1 (Pin_1), J?.23 (Pin_23)
- net GPIO3 is gone; now on net GPIO6: J112.2 (Pin_2), J?.31 (Pin_31)
- net GPIO11: no longer J112.3 (Pin_3), J?.26 (Pin_26)
- net GPIO19: now also J112.4 (Pin_4), J?.35 (Pin_35); no longer J112.6 (Pin_6), J?.37 (Pin_37)
- net GPIO6: no longer J112.4 (Pin_4), J?.35 (Pin_35)
- new net GPIO26: J112.6 (Pin_6), J?.37 (Pin_37)
- new net GPIO7: J112.3 (Pin_3), J?.26 (Pin_26)
Changed lines of the file:
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@@
     (effects (font (size 1.27 1.27) (color 0 132 0 1)) (justify left bottom))
   )
-  (label "GPIO3" (at 34.29 123.19 0) (fields_autoplaced)
+  (label "GPIO6" (at 34.29 123.19 0) (fields_autoplaced)
     (effects (font (size 1.27 1.27)) (justify left bottom))
   )
@@
     (effects (font (size 1.27 1.27) (color 0 1 255 1)) (justify left bottom))
   )
-  (label "GPIO6" (at 34.29 128.27 0) (fields_autoplaced)
+  (label "GPIO19" (at 34.29 128.27 0) (fields_autoplaced)
     (effects (font (size 1.27 1.27)) (justify left bottom))
     (property "info" "pwm" (at 34.29 129.54 0)
@@
     (effects (font (size 1.27 1.27) (color 0 1 255 1)) (justify right bottom))
   )
-  (label "GPIO3" (at 228.6 29.21 180) (fields_autoplaced)
+  (label "GPIO6" (at 228.6 29.21 180) (fields_autoplaced)
     (effects (font (size 1.27 1.27)) (justify right bottom))
   )
@@
     (effects (font (size 1.27 1.27) (color 0 132 0 1)) (justify left bottom))
   )
-  (label "GPIO11" (at 93.98 115.57 180) (fields_autoplaced)
+  (label "GPIO7" (at 93.98 115.57 180) (fields_autoplaced)
     (effects (font (size 1.27 1.27)) (justify right bottom))
   )
@@
     (effects (font (size 1.27 1.27) (color 250 26 255 1)) (justify left bottom))
   )
-  (label "GPIO6" (at 228.6 34.29 180) (fields_autoplaced)
+  (label "GPIO19" (at 228.6 34.29 180) (fields_autoplaced)
     (effects (font (size 1.27 1.27)) (justify right bottom))
   )
@@
     (effects (font (size 1.27 1.27) (color 255 2 4 1)) (justify right bottom))
   )
-  (label "GPIO19" (at 34.29 130.81 0) (fields_autoplaced)
+  (label "GPIO26" (at 34.29 130.81 0) (fields_autoplaced)
     (effects (font (size 1.27 1.27)) (justify left bottom))
     (property "info" "pwm" (at 34.29 132.08 0)
@@
     (effects (font (size 1.27 1.27) (color 0 132 0 1)) (justify left bottom))
   )
-  (label "GPIO19" (at 228.6 39.37 180) (fields_autoplaced)
+  (label "GPIO26" (at 228.6 39.37 180) (fields_autoplaced)
     (effects (font (size 1.27 1.27)) (justify right bottom))
   )
@@
     (effects (font (size 1.27 1.27) (color 255 0 139 1)) (justify left bottom))
   )
-  (label "GPIO11" (at 228.6 31.75 180) (fields_autoplaced)
+  (label "GPIO7" (at 228.6 31.75 180) (fields_autoplaced)
     (effects (font (size 1.27 1.27)) (justify right bottom))
   )
@@
     (effects (font (size 1.27 1.27) (color 255 2 4 1)) (justify left bottom))
   )
-  (label "GPIO2" (at 34.29 113.03 0) (fields_autoplaced)
+  (label "GPIO11" (at 34.29 113.03 0) (fields_autoplaced)
     (effects (font (size 1.27 1.27)) (justify left bottom))
   )
@@
     (effects (font (size 1.27 1.27) (color 255 115 25 1)) (justify left bottom))
   )
-  (label "GPIO2" (at 228.6 26.67 180) (fields_autoplaced)
+  (label "GPIO11" (at 228.6 26.67 180) (fields_autoplaced)
     (effects (font (size 1.27 1.27)) (justify right bottom))
   )

Commit message: finalize pcb
Connections:
- net +3.3V: now also J114.5 (Pin_5); no longer J114.1 (Pin_1)
- net 5.1V: now also J114.2 (Pin_2); no longer J114.4 (Pin_4)
- net GND: now also J114.1 (Pin_1), J114.4 (Pin_4); no longer J114.2 (Pin_2), J114.5 (Pin_5)
Other:
- moved on the sheet: J114, J115

Commit message: add picture
Other:
- company: (none) -> Ares ENSEA
- title: (none) -> Carte de commande Coupe de France de Robotique 2024
Changed lines of the file:
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@@
 (kicad_sch (version 20230121) (generator eeschema)
   (paper "A4")
+  (title_block
+    (title "Carte de commande Coupe de France de Robotique 2024")
+    (date "2024-01-30")
+    (company "Ares ENSEA")
+  )
   (junction (at 58.42 33.02) (diameter 0) (color 0 0 0 0)
   )
@@
     (stroke (width 0) (type default))
   )
+  (wire (pts (xy 272.7718 91.44) (xy 269.24 91.44))
+    (stroke (width 0) (type default))
+  )
   (wire (pts (xy 208.28 45.72) (xy 208.28 44.45))
     (stroke (width 0) (type default))
@@
     (stroke (width 0) (type default))
   )
+  (wire (pts (xy 272.7718 91.4793) (xy 272.7718 91.44))
+    (stroke (width 0) (type default))
+  )
   (wire (pts (xy 170.18 33.02) (xy 170.18 36.83))
     (stroke (width 0) (type default))
@@
   )
   (wire (pts (xy 121.92 151.13) (xy 121.92 157.48))
-    (stroke (width 0) (type default))
-  )
-  (wire (pts (xy 269.24 91.44) (xy 276.86 91.44))
     (stroke (width 0) (type default))
   )
@@
     (effects (font (size 1.27 1.27)) (justify left bottom))
   )
-  (text "Connecteur de lien avec la RasberryPi" (at 14.986 66.802 0)
+  (text "Connecteur de lien avec la RasberryPi" (at 31.4876 74.335 0)
     (effects (font (size 1.27 1.27)) (justify left bottom))
   )
@@
     )
   )
-  (symbol (lib_id "power:+3.3V") (at 276.86 91.44 270) (unit 1)
-    (in_bom yes) (on_board yes) (dnp no) (fields_autoplaced)
-    (property "Reference" "#PWR0130" (at 273.05 91.44 0)
-      (effects (font (size 1.27 1.27)) hide)
-    )
-    (property "Value" "+3.3V" (at 280.67 91.44 90)
-      (effects (font (size 1.27 1.27)) (justify left))
-    )
-    (property "Footprint" "" (at 276.86 91.44 0)
-      (effects (font (size 1.27 1.27)) hide)
-    )
-    (property "Datasheet" "" (at 276.86 91.44 0)
-      (effects (font (size 1.27 1.27)) hide)
-    )
+  (symbol (lib_id "power:+3.3V") (at 272.7718 91.4793 270) (unit 1)
+    (in_bom yes) (on_board yes) (dnp no) (fields_autoplaced)
+    (property "Reference" "#PWR0130" (at 268.9618 91.4793 0)
+      (effects (font (size 1.27 1.27)) hide)
+    )
+    (property "Value" "+3.3V" (at 276.5818 91.4793 90)
+      (effects (font (size 1.27 1.27)) (justify left))
+    )
+    (property "Footprint" "" (at 272.7718 91.4793 0)
+      (effects (font (size 1.27 1.27)) hide)
+    )
+    (property "Datasheet" "" (at 272.7718 91.4793 0)
+      (effects (font (size 1.27 1.27)) hide)
+    )

Commit message: update pcb
Parts:
- added R1, R3: 2k7, Resistor_SMD:R_0402_1005Metric, symbol Device:R_Small
- added R2, R4: 3k3, Resistor_SMD:R_0402_1005Metric, symbol Device:R_Small
Connections:
- net +3.3V: no longer J113.7 (Pin_7), J113.8 (Pin_8)
- net 7.4V: now also J113.7 (Pin_7), J113.8 (Pin_8)
- net GND: now also R2.2, R4.2
- net GPIO20: now also R3.2, R4.1; no longer J112.7 (Pin_7)
- net GPIO21: now also R1.2, R2.1; no longer J112.8 (Pin_8)
- new net: J112.7 (Pin_7), R3.1
- new net: J112.8 (Pin_8), R1.1
Other:
- moved on the sheet: H?
