File: 1A/PAMI/PCB/PAMI_mb/PAMI_mb.kicad_sch (KiCad schematic)
At the start: 21 parts, among them J101 Conn_ST_STDC14, J102 Conn_02x20_Odd_Even, J103 Conn_01x04, J104 Conn_01x04, U101 STM32G431KBTx, U102 LT1076CR-PBF, U103 AZ1117-3.3

Commit message: add datasheets
Parts:
- added C1, C2, C3: 100n, symbol Device:C_Small
- added R1, R3: 4k7, symbol Device:R_Small
- added R2, R4: 100, symbol Device:R_Small
- added R5: 10k, symbol Device:R_Small
- added SW1, SW2, SW3: SW_Push, symbol Switch:SW_Push
- C105: MFR 865060445005 -> (none); MPN (none) -> 865060445005
- CR101: MPN (none) -> DST10100S
Connections:
- net +3.3V: now also R1.1, R3.1
- net GND: now also C3.2, R2.2, R4.2, R5.2, SW1.1, SW2.1, SW3.1
- net at U101.31 (PB8): now also R5.1
- net NRST: now reaches U101.4 (PG10)
- net NRST: now also J101.12 (~{RST}), C3.1, SW3.2
- net +5.1V renamed +5V
- new net: C1.2, R2.1
- new net: C2.2, R4.1
- new net BTN_1: C1.1, R1.2, SW1.2
- new net BTN_2: C2.1, R3.2, SW2.2
Other:
- sheet TMC2225 renamed TMC2225-1
- sheet TMC2226 renamed TMC2225-2
- moved on the sheet: C101, C102, C103, C104, J101

Commit message: update PAMI pcb
Parts:
- removed C1, C2, C3: 100n, symbol Device:C_Small
- removed D101: LED, LED_SMD:LED_0603_1608Metric, symbol Device:LED
- removed R104: 1k, Resistor_SMD:R_0402_1005Metric, symbol Device:R_Small
- removed SW1, SW2: SW_Push, symbol Switch:SW_Push
- added C10, C5, C6, C9: 10n, Capacitor_SMD:C_0402_1005Metric_Pad0.74x0.62mm_HandSolder, symbol Device:C_Small
- added C11, C12: 1u, Capacitor_SMD:C_0402_1005Metric_Pad0.74x0.62mm_HandSolder, symbol Device:C_Small
- added C16, C17: 10u, Capacitor_SMD:CP_Elec_6.3x5.4, symbol Device:C_Polarized_Small
- added C35, C7: 100n, Capacitor_SMD:C_0402_1005Metric_Pad0.74x0.62mm_HandSolder, symbol Device:C_Small
- added C8: 10u, Capacitor_SMD:CP_Elec_4x5.4, symbol Device:C_Polarized_Small
- added D1: LED_RED, LED_SMD:LED_0603_1608Metric, symbol Device:LED
- added D2, D3, D4, D5: LED_GREEN, LED_SMD:LED_0603_1608Metric_Pad1.05x0.95mm_HandSolder, symbol Device:LED
- added D6, D7, D8, D9: LED_RED, LED_SMD:LED_0603_1608Metric_Pad1.05x0.95mm_HandSolder, symbol Device:LED
- added H1, H2, H3, H4: MountingHole_Pad, MountingHole:MountingHole_2.7mm_M2.5_DIN965_Pad, symbol Mechanical:MountingHole_Pad
- added J3: Battery, custom:691322110002, symbol Connector_Generic:Conn_01x02
- added J4: Charge, custom:691322110002, symbol Connector_Generic:Conn_01x02
- added J5: Stop, custom:691322110002, symbol Connector_Generic:Conn_01x02
- added J6: Conn_01x05, symbol Connector_Generic:Conn_01x05
- added J7: 173010542, libs:173010542_5V_Buck, symbol 173010542_5V_Buck:173010542
- added J8, J9: Conn_01x04, Connector_JST:JST_XH_B4B-XH-A_1x04_P2.50mm_Vertical, symbol Connector_Generic:Conn_01x04
- added R10, R19, R6, R8: 1k6, Resistor_SMD:R_0402_1005Metric_Pad0.72x0.64mm_HandSolder, symbol Device:R_Small
- added R11, R12, R31, R7, R9: 10k, Resistor_SMD:R_0402_1005Metric_Pad0.72x0.64mm_HandSolder, symbol Device:R_Small
- added R13: 5k6, Resistor_SMD:R_0402_1005Metric_Pad0.72x0.64mm_HandSolder, symbol Device:R_Small
- added R15, R18: 3k6, Resistor_SMD:R_0402_1005Metric_Pad0.72x0.64mm_HandSolder, symbol Device:R_Small
- added R30: 15k, Resistor_SMD:R_0402_1005Metric_Pad0.72x0.64mm_HandSolder, symbol Device:R_Small
- added SW1: SW_Push_SPDT, symbol Switch:SW_Push_SPDT
- added SW2: RotaryEncoder_Switch, symbol Device:RotaryEncoder_Switch
- added TP1: TestPoint, Connector_Pin:Pin_D0.9mm_L10.0mm_W2.4mm_FlatFork, symbol Connector:TestPoint
- C1: renamed from C101; footprint (none) -> Capacitor_SMD:C_0402_1005Metric_Pad0.74x0.62mm_HandSolder
- C13: renamed from C106; footprint Capacitor_SMD:C_0402_1005Metric -> Capacitor_SMD:C_0402_1005Metric_Pad0.74x0.62mm_HandSolder
- C14: renamed from C105; MFR (none) -> 865060445005; MPN 865060445005 -> (none)
- C2: renamed from C102; footprint (none) -> Capacitor_SMD:C_0402_1005Metric_Pad0.74x0.62mm_HandSolder
- C3: renamed from C103; footprint (none) -> Capacitor_SMD:C_0402_1005Metric_Pad0.74x0.62mm_HandSolder
- C4: renamed from C104; footprint (none) -> Capacitor_SMD:C_0402_1005Metric_Pad0.74x0.62mm_HandSolder
- CR1: renamed from CR101; MPN DST10100S -> (none)
- J10: renamed from J103; footprint (none) -> Connector_JST:JST_XH_B4B-XH-A_1x04_P2.50mm_Vertical
- J11: renamed from J104; footprint (none) -> Connector_JST:JST_XH_B4B-XH-A_1x04_P2.50mm_Vertical
- J2: renamed from J101; footprint (none) -> Connector_PinHeader_1.27mm:PinHeader_2x07_P1.27mm_Vertical_SMD
- R1: value 4k7 -> 100k; footprint (none) -> Resistor_SMD:R_0402_1005Metric_Pad0.72x0.64mm_HandSolder
- R14: renamed from R101; footprint Resistor_SMD:R_0402_1005Metric -> Resistor_SMD:R_0402_1005Metric_Pad0.72x0.64mm_HandSolder
- R16: renamed from R102; footprint Resistor_SMD:R_0402_1005Metric -> Resistor_SMD:R_0402_1005Metric_Pad0.72x0.64mm_HandSolder
- R17: renamed from R103; footprint Resistor_SMD:R_0402_1005Metric -> Resistor_SMD:R_0402_1005Metric_Pad0.72x0.64mm_HandSolder
- R2: value 100 -> 560; footprint (none) -> Resistor_SMD:R_0402_1005Metric_Pad0.72x0.64mm_HandSolder
- R3: value 4k7 -> 1k6; footprint (none) -> Resistor_SMD:R_0402_1005Metric_Pad0.72x0.64mm_HandSolder
- R4: value 100 -> 10k; footprint (none) -> Resistor_SMD:R_0402_1005Metric_Pad0.72x0.64mm_HandSolder
- R5: footprint (none) -> Resistor_SMD:R_0402_1005Metric_Pad0.72x0.64mm_HandSolder
- U3: renamed from U103; value AZ1117-3.3 -> AZ1117CH2-3.3TRG1; MPN (none) -> AZ1117CH2-3.3TRG1
- renumbered C107 to C15, J102 to J1, L101 to L1, U101 to U1, U102 to U2
Connections:
- net BTN_1 is gone; now on net GND: R1.2
- net +3.3V: now also J1.1 (Pin_1), U3.2 (VO), C12.1, C17.1, C7.2, J9.2 (Pin_2), R11.1, R19.1, R7.2, R9.2; no longer R1.1, R3.1
- net +5V: now also U3.3 (VI), C11.1, C16.1, J7.3 (VOUT), J8.4 (Pin_4), R15.1; no longer C15.1, L1.2, R16.1
- net GND: now also J1.11 (Pin_11), J1.20 (Pin_20), J1.25 (Pin_25), J1.30 (Pin_30), J1.39 (Pin_39), J1.6 (Pin_6), SW3.2, U3.1 (GND), C10.2, C11.2, C12.2, C16.2, C17.2, C35.2, C5.2, C6.2, C7.1, C8.2, C9.2, D1.1 (K), D2.1 (K), D3.1 (K), D4.1 (K), D5.1 (K), D6.1 (K), D7.1 (K), D8.1 (K), D9.1 (K), H1.1, H2.1, H3.1, H4.1, J3.1 (Pin_1), J4.1 (Pin_1), J6.1 (Pin_1), J7.2 (GND), J8.1 (Pin_1), J9.1 (Pin_1), R31.2, SW2.C, SW2.S2; no longer R2.2, R4.2, R5.2, SW3.1
- net NRST: now also SW3.1, C9.1; no longer SW3.2
- net STLINK_RX: now also U1.27 (PB4); no longer U1.8 (PA3)
- net STLINK_TX: now also U1.26 (PB3); no longer U1.25 (PA15)
- net VCC: now also C8.1, J5.2 (Pin_2), J7.1 (VIN), R13.1, R30.1, TP1.1
- net VFB: now reaches R16.2, R17.1, U2.5 (FB)
- net ENCODEUR_B: now reaches R5.1
- net ENCODEUR_B: now also U1.19 (PA9), C5.1; no longer U1.31 (PB8)
- net V_CHARGE: now reaches R2.1
- net V_CHARGE: now also J4.2 (Pin_2), SW1.3 (C)
- net ENCODEUR_A: now reaches R4.1
- net ENCODEUR_A: now also U1.18 (PA8), C6.1
- net PWM_MOTOR_R_TIM3_CH1: now reaches U1.11 (PA6)
- net DIR_MOTOR_R: now reaches U1.12 (PA7)
- net ENCODEUR_BTN: now reaches U1.13 (PB0)
- net ENCODEUR_BTN: now also C10.1, R12.2
- net PF0_LED1: now reaches U1.2 (PF0)
- net PF0_LED1: now also J6.3 (Pin_3), R6.1
- net RASPBERRY_PI_RX: now reaches U1.20 (PA10)
- net RASPBERRY_PI_RX: now also J1.10 (Pin_10)
- net PA11_USR_BTN_1: now reaches U1.21 (PA11)
- net PA12_USR_BTN_2: now reaches U1.22 (PA12)
- net PB5_LED3: now reaches U1.28 (PB5)
- net PB5_LED3: now also J6.5 (Pin_5), R10.1
- net RASPBERRY_PI_TX: now reaches U1.29 (PB6)
- net RASPBERRY_PI_TX: now also J1.8 (Pin_8)
- net PF1_LED2: now reaches U1.3 (PF1)
- net PF1_LED2: now also J6.4 (Pin_4), R8.1
- net I2C_SDA: now reaches U1.30 (PB7)
- net I2C_SDA: now also J9.4 (Pin_4)
- net ADC_BATT: now reaches U1.5 (PA0)
- net ADC_BATT: now also C35.1, R30.2, R31.1
- net PA1_USR_BTN_0: now reaches U1.6 (PA1)
- net LIDAR_LP_TX: now reaches U1.7 (PA2)
- net LIDAR_LP_TX: now also J8.2 (Pin_2)
- net DIR_MOTOR_L: now reaches U1.9 (PA4)
- net +5.1V: now reaches J1.2 (Pin_2)
- net +5.1V: now also C15.1, J1.4 (Pin_4), L1.2, R16.1, R18.1
- net BTN_2: no longer names the net of R3.2
- net BTN_2: now also D2.2 (A)
- net PWM_MOTOR_L_TIM_CH1 renamed PWM_MOTOR_L_TIM2_CH1
- new net: R5.2, R7.1, SW2.B
- new net: D3.2 (A), R6.2
- new net: D8.2 (A), R18.2
- new net: J5.1 (Pin_1), SW1.1 (A)
- new net: R4.2, R9.1, SW2.A
- new net: D6.2 (A), R13.2
- new net: D7.2 (A), R15.2
- new net: R11.2, R12.1, SW2.S1
- new net: D4.2 (A), R8.2
- new net: D5.2 (A), R10.2
- new net: D9.2 (A), R19.2
- new net: D1.2 (A), R2.2
- new net I2C_SCL: J9.3 (Pin_3), U1.25 (PA15)
- new net LIDAR_LP_RX: J8.3 (Pin_3), U1.8 (PA3)
- new net PB8-BOOT0_LED0: J6.2 (Pin_2), R1.1, R3.1, U1.31 (PB8)
- new net V_BAT: J3.2 (Pin_2), SW1.2 (B)
- no-connect marks 4 -> 33
Other:
- sheet TMC2225-1 renamed TMC2225
- sheet TMC2225-2 renamed TMC2226
- added sheet GPIO_Filter (GPIO_Filter.kicad_sch)
- added sheet GPIO_Filter1 (GPIO_Filter.kicad_sch)
- added sheet GPIO_Filter2 (GPIO_Filter.kicad_sch)
- note added: "100n for power filtering, 1 by VDD/VDDA pin"
- note added: "BUCK Regalator Based on LT1076CR 5.1 for RPI Max : 2A"
- note added: "BUCK Regalator Based on Wurth 173010542 5V for LIDAR Vin : 7V-42V Vout : 5V Max : 1A"
- note added: "Buttons"
- note added: "Connector for LIDAR"
- note added: "Connector for OLED Screen"
- note added: "Green LED 3.2V @ 20mA max R for 2mA @ 2.5V"
- note added: "LDO Regalator Based on AZ1117CH2-3.3TRG1 3.3V for MCU and others Max : 1.35A"
- note added: "MCU"
- note added: "Motor Drivers"
- note added: "Mounting holes"
- note added: "Pull-down for booting from Flash Memory"
- note added: "RED LED 2V @ 20mA max R for 10mA @ 1.8V"
- note added: "RED LED 2V @ 20mA max R for 1mA @ 1.6V"
- note added: "RaspberryPi Connector"
- note added: "Reference voltage VFB = 2.21V"
- note added: "Rotary Enc Button"
- note added: "https://fr.rs-online.com/web/p/blocs-batteries-rechargeables/7770406 Battery, 6 cell NIMH 7.2V, 2Ah RS ref : 777-0406"
- note removed: "Reference voltage : VFB = 2.21V"
- note removed: "Rpi Connector"
- note removed: "Wurth 173010542 Buck 5V"
- title: (none) -> PAMI - CFR 2024
- moved on the sheet: C1, C13, C14, C15, C2, C3, C4, J1, J10, J11, J2, L1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
