File: 1A/PAMI/PCB/PAMI_mb/TMC2225.kicad_sch (KiCad schematic)
At the start: 0 parts

Commit message: update PAMI pcb
Parts:
- added C18: 100u, Capacitor_SMD:C_0402_1005Metric_Pad0.74x0.62mm_HandSolder, symbol Device:C_Polarized_Small
- added C19, C20, C22, C24: 100n, Capacitor_SMD:C_0402_1005Metric_Pad0.74x0.62mm_HandSolder, symbol Device:C_Small
- added C21: 22n, Capacitor_SMD:C_0402_1005Metric_Pad0.74x0.62mm_HandSolder, symbol Device:C_Small
- added C23: 22u, symbol Device:C_Small
- added R20: Rsa, symbol Device:R_Small
- added R21: Rsb, symbol Device:R_Small
- added U4: TMC2225-SA, symbol TMC2225:TMC2225-SA
Connections:
- net 3.3V: now also C24.1, U4.16 (VCC_IO), U4.17 (PDN_UART), U4.19 (SPREAD), U4.25 (MS1), U4.26 (MS2)
- net DIR: now also U4.20 (DIR)
- net OA1: now also U4.7 (OA1)
- net OA2: now also U4.5 (OA2)
- net OB1: now also U4.8 (OB1)
- net OB2: now also U4.10 (OB2)
- net PWM: now also U4.22 (STEP)
- new net: R21.2, U4.9 (BRB)
- new net: C23.1, U4.15 (5VOUT)
- new net: R20.2, U4.6 (BRA)
- new net: C22.2, U4.1 (CPO)
- new net: C22.1, U4.2 (CPI)
- new net: C21.2, U4.3 (VCP)
- new net GND: C18.2, C19.1, C20.1, C23.2, C24.2, R20.1, R21.1, U4.12 (VREF), U4.13 (TEST), U4.14 (GND), U4.21 (ENN), U4.24 (CLK), U4.28 (GND), U4.EPAD (GROUND)
- new net VCC: C18.1, C19.2, C20.2, C21.1, U4.11 (VS), U4.4 (VS)
- no-connect marks 0 -> 2
