File: 1A/PAMI/PCB/PCB_Projet_v2/GPIO_Filter.kicad_sch (KiCad schematic)
At the start: 4 parts, among them SW4 SW_Push

Commit message: update pcb
Parts:
- C25: footprint Capacitor_SMD:C_0603_1608Metric -> Capacitor_SMD:C_0402_1005Metric
- SW4: footprint Button_Switch_THT:SW_PUSH_6mm -> Button_Switch_SMD:SW_Push_1P1T_NO_6x6mm_H9.5mm

Commit message: update PAMI pcb
Parts:
- renumbered C25 to C401, R35 to R401, R36 to R402, SW4 to SW401
Changed lines of the file:
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@@
 		(on_board yes)
 		(dnp no)
-		(property "Reference" "#PWR078"
+		(property "Reference" "#PWR0401"
 			(at 132.08 111.76 0)
 			(effects
@@
 			(project "PAMI_mb"
 				(path "/bb3e6145-6642-4de1-802f-741b252e53ea/b74b7472-b7d2-4b72-8a8d-d152a9cce4ed"
-					(reference "#PWR078")
-					(unit 1)
-				)
-				(path "/bb3e6145-6642-4de1-802f-741b252e53ea/e35bafc9-e0aa-4431-83a8-584d217afb21"
-					(reference "#PWR079")
-					(unit 1)
-				)
-				(path "/bb3e6145-6642-4de1-802f-741b252e53ea/f5d83293-9460-4743-be34-e43aa5f52b77"
-					(reference "#PWR080")
+					(reference "#PWR0401")
+					(unit 1)
+				)
+				(path "/bb3e6145-6642-4de1-802f-741b252e53ea/e35bafc9-e0aa-4431-83a8-584d217afb21"
+					(reference "#PWR0501")
+					(unit 1)
+				)
+				(path "/bb3e6145-6642-4de1-802f-741b252e53ea/f5d83293-9460-4743-be34-e43aa5f52b77"
+					(reference "#PWR0601")
 					(unit 1)
 				)
@@
 		(on_board yes)
 		(dnp no)
-		(property "Reference" "R36"
+		(property "Reference" "R402"
 			(at 143.51 92.71 90)
 			(effects
@@
 			(project "PAMI_mb"
 				(path "/bb3e6145-6642-4de1-802f-741b252e53ea/b74b7472-b7d2-4b72-8a8d-d152a9cce4ed"
-					(reference "R36")
-					(unit 1)
-				)
-				(path "/bb3e6145-6642-4de1-802f-741b252e53ea/f5d83293-9460-4743-be34-e43aa5f52b77"
-					(reference "R40")
-					(unit 1)
-				)
-				(path "/bb3e6145-6642-4de1-802f-741b252e53ea/e35bafc9-e0aa-4431-83a8-584d217afb21"
-					(reference "R38")
+					(reference "R402")
+					(unit 1)
+				)
+				(path "/bb3e6145-6642-4de1-802f-741b252e53ea/f5d83293-9460-4743-be34-e43aa5f52b77"
+					(reference "R602")
+					(unit 1)
+				)
+				(path "/bb3e6145-6642-4de1-802f-741b252e53ea/e35bafc9-e0aa-4431-83a8-584d217afb21"
+					(reference "R502")
 					(unit 1)
 				)
@@
 		(on_board yes)
 		(dnp no)
-		(property "Reference" "R35"
+		(property "Reference" "R401"
 			(at 133.35 90.17 0)
 			(effects
@@
 			(project "PAMI_mb"
 				(path "/bb3e6145-6642-4de1-802f-741b252e53ea/b74b7472-b7d2-4b72-8a8d-d152a9cce4ed"
-					(reference "R35")
-					(unit 1)
-				)
-				(path "/bb3e6145-6642-4de1-802f-741b252e53ea/f5d83293-9460-4743-be34-e43aa5f52b77"
-					(reference "R39")
-					(unit 1)
-				)
-				(path "/bb3e6145-6642-4de1-802f-741b252e53ea/e35bafc9-e0aa-4431-83a8-584d217afb21"
-					(reference "R37")
+					(reference "R401")
+					(unit 1)
+				)
+				(path "/bb3e6145-6642-4de1-802f-741b252e53ea/f5d83293-9460-4743-be34-e43aa5f52b77"
+					(reference "R601")
+					(unit 1)
+				)
+				(path "/bb3e6145-6642-4de1-802f-741b252e53ea/e35bafc9-e0aa-4431-83a8-584d217afb21"
+					(reference "R501")
 					(unit 1)
 				)
@@
 		(dnp no)
 		(fields_autoplaced yes)
-		(property "Reference" "C25"
+		(property "Reference" "C401"
 			(at 134.874 96.5263 0)
 			(effects
@@
 			(project "PAMI_mb"
 				(path "/bb3e6145-6642-4de1-802f-741b252e53ea/b74b7472-b7d2-4b72-8a8d-d152a9cce4ed"
-					(reference "C25")
-					(unit 1)
-				)
-				(path "/bb3e6145-6642-4de1-802f-741b252e53ea/f5d83293-9460-4743-be34-e43aa5f52b77"
-					(reference "C27")
-					(unit 1)
-				)
-				(path "/bb3e6145-6642-4de1-802f-741b252e53ea/e35bafc9-e0aa-4431-83a8-584d217afb21"
-					(reference "C26")
+					(reference "C401")
+					(unit 1)
+				)
+				(path "/bb3e6145-6642-4de1-802f-741b252e53ea/f5d83293-9460-4743-be34-e43aa5f52b77"
+					(reference "C601")
+					(unit 1)
+				)
+				(path "/bb3e6145-6642-4de1-802f-741b252e53ea/e35bafc9-e0aa-4431-83a8-584d217afb21"
+					(reference "C501")
 					(unit 1)
 				)
@@
 		(dnp no)
 		(fields_autoplaced yes)
-		(property "Reference" "SW4"
+		(property "Reference" "SW401"
 			(at 160.02 96.52 90)
 			(effects
@@
 			(project "PAMI_mb"
 				(path "/bb3e6145-6642-4de1-802f-741b252e53ea/b74b7472-b7d2-4b72-8a8d-d152a9cce4ed"
-					(reference "SW4")
-					(unit 1)
-				)
-				(path "/bb3e6145-6642-4de1-802f-741b252e53ea/e35bafc9-e0aa-4431-83a8-584d217afb21"
-					(reference "SW5")
-					(unit 1)
-				)
-				(path "/bb3e6145-6642-4de1-802f-741b252e53ea/f5d83293-9460-4743-be34-e43aa5f52b77"
-					(reference "SW6")
-					(unit 1)
-				)
+					(reference "SW401")
+					(unit 1)
+				)
+				(path "/bb3e6145-6642-4de1-802f-741b252e53ea/e35bafc9-e0aa-4431-83a8-584d217afb21"
+					(reference "SW501")
+					(unit 1)
+				)
+				(path "/bb3e6145-6642-4de1-802f-741b252e53ea/f5d83293-9460-4743-be34-e43aa5f52b77"
+					(reference "SW601")
+					(unit 1)
+				)
